Commit message: modelo spider

File: install/spider_description/share/spider_description/urdf/spider.urdf.xacro (robot description, xacro)
@@ -2,14 +2,37 @@
 <robot xmlns:xacro="http://www.ros.org/wiki/xacro" name="spider">
   <!-- ============================================================
-       SPIDER QUADRUPED ROBOT - URDF/XACRO
-       Hito 1: Structural model for Ignition Gazebo 6 / ROS2 Humble
-       4 legs in X-pattern: front_right(45°), front_left(135°),
-                             back_left(-135°), back_right(-45°)
-       3 DOF per leg: coxa(Z), femur(Y), tibia(Y)
-  ============================================================ -->
-  <!-- ============================================================
-       INERTIA MACROS (analytic formulas for primitives)
-  ============================================================ -->
-  <!-- Solid sphere: Ixx=Iyy=Izz = 2/5 * m * r^2 -->
+       SPIDER QUADRUPED ROBOT - URDF/XACRO  (Hito 1 rev.2)
+       Body: flat base cylinder + dome sphere (no leg intersection)
+       4 legs in X-pattern at 45°/135°/-135°/-45°
+       3 DOF per leg: coxa(Z) → femur(Y) → tibia(Y)
+  ============================================================ -->
+  <!-- ============================================================
+       CONSTANTS
+  ============================================================ -->
+  <!-- Body geometry -->
+  <xacro:property name="base_r"        value="0.13"/>   <!-- base disc radius -->
+  <xacro:property name="base_h"        value="0.025"/>  <!-- base disc height -->
+  <xacro:property name="dome_r"        value="0.10"/>   <!-- dome sphere radius -->
+  <!-- dome center is at z = base_h/2 + dome_r*0.45 so it sits on top of base -->
+  <xacro:property name="dome_z"        value="0.06"/>
+  <!-- Hip attachment: on top surface of base disc, at radial distance hip_r -->
+  <xacro:property name="hip_r"         value="0.10"/>   <!-- radial offset of coxa joint from centre -->
+  <xacro:property name="hip_z_offset"  value="0.0125"/> <!-- = base_h/2, top of base disc -->
+  <!-- Leg geometry -->
+  <xacro:property name="coxa_r"  value="0.018"/>
+  <xacro:property name="coxa_l"  value="0.045"/>
+  <xacro:property name="femur_r" value="0.014"/>
+  <xacro:property name="femur_l" value="0.10"/>
+  <xacro:property name="tibia_r" value="0.012"/>
+  <xacro:property name="tibia_l" value="0.13"/>
+  <!-- Masses (total body = 1.5 kg) -->
+  <xacro:property name="base_mass"  value="1.5"/>
+  <xacro:property name="coxa_mass"  value="0.06"/>
+  <xacro:property name="femur_mass" value="0.12"/>
+  <xacro:property name="tibia_mass" value="0.08"/>
+  <!-- ============================================================
+       INERTIA MACROS
+  ============================================================ -->
+  <!-- Solid sphere -->
   <xacro:macro name="sphere_inertia" params="m r">
     <inertial>
@@ -23,5 +46,5 @@
     </inertial>
   </xacro:macro>
-  <!-- Solid cylinder (axis Z): Ixx=Iyy = m*(3r^2+l^2)/12  Izz = m*r^2/2 -->
+  <!-- Solid cylinder (symmetry axis = Z) -->
   <xacro:macro name="cylinder_inertia" params="m r l">
     <inertial>
@@ -35,111 +58,137 @@
     </inertial>
   </xacro:macro>
+  <!-- Composite inertia for base_link:
+       Modelled as a thick disc (dominant contributor).
+       CoM placed at z=0 (centre of the disc).
+       base_r=0.13  base_h=0.025  m=1.5 kg
+       Ixx=Iyy = m*(3r²+h²)/12  Izz = m*r²/2  -->
+  <xacro:macro name="base_link_inertia">
+    <inertial>
+      <origin xyz="0 0 0" rpy="0 0 0"/>
+      <mass value="${base_mass}"/>
+      <inertia
+        ixx="${base_mass * (3*base_r*base_r + base_h*base_h) / 12.0}"
+        iyy="${base_mass * (3*base_r*base_r + base_h*base_h) / 12.0}"
+        izz="${base_mass * base_r*base_r / 2.0}"
+        ixy="0" ixz="0" iyz="0"/>
+    </inertial>
+  </xacro:macro>
   <!-- ============================================================
        LEG MACRO
-       Parameters:
-         leg_name  - identifier (front_right, front_left, back_left, back_right)
-         hip_x     - X position of coxa joint on base sphere surface
-         hip_y     - Y position of coxa joint on base sphere surface
-         hip_z     - Z position of coxa joint (0 = equator of sphere)
-         hip_yaw   - Initial rotation of the coxa around Z (for visual alignment)
-  ============================================================ -->
-  <xacro:macro name="leg" params="leg_name hip_x hip_y hip_z hip_yaw">
-    <!-- COXA LINK -->
-    <!-- Cylinder r=0.02 l=0.06, mass=0.08 kg, axis along Z of joint -->
+       hip_x, hip_y : position of the coxa joint in base_link frame
+                       (on top surface of base disc, at the edge)
+       hip_yaw       : yaw angle so coxa extends radially outward
+  ============================================================ -->
+  <xacro:macro name="leg" params="leg_name hip_x hip_y hip_yaw">
+    <!-- ── COXA LINK ─────────────────────────────────────────────
+         Small cylinder representing the hip servo block.
+         Oriented radially (axis along X of joint frame).
+         Visual/collision centre at x=coxa_l/2 from joint origin.
+    ─────────────────────────────────────────────────────────── -->
     <link name="${leg_name}_coxa_link">
-      <xacro:cylinder_inertia m="0.08" r="0.02" l="0.06"/>
+      <!-- Inertia: cylinder with axis along X → rotate cylinder_inertia 90° about Y.
+           For a cylinder with axis along X: Ixx=m*r²/2  Iyy=Izz=m*(3r²+l²)/12 -->
+      <inertial>
+        <origin xyz="${coxa_l/2} 0 0" rpy="0 0 0"/>
+        <mass value="${coxa_mass}"/>
+        <inertia
+          ixx="${coxa_mass * coxa_r*coxa_r / 2.0}"
+          iyy="${coxa_mass * (3*coxa_r*coxa_r + coxa_l*coxa_l) / 12.0}"
+          izz="${coxa_mass * (3*coxa_r*coxa_r + coxa_l*coxa_l) / 12.0}"
+          ixy="0" ixz="0" iyz="0"/>
+      </inertial>
       <visual>
-        <origin xyz="0 0 0.03" rpy="0 0 0"/>
-        <geometry>
-          <cylinder radius="0.02" length="0.06"/>
-        </geometry>
-        <material name="dark_gray">
-          <color rgba="0.3 0.3 0.3 1.0"/>
-        </material>
+        <origin xyz="${coxa_l/2} 0 0" rpy="0 ${pi/2} 0"/>
+        <geometry><cylinder radius="${coxa_r}" length="${coxa_l}"/></geometry>
+        <material name="servo_blue"><color rgba="0.2 0.35 0.75 1.0"/></material>
       </visual>
       <collision>
-        <origin xyz="0 0 0.03" rpy="0 0 0"/>
-        <geometry>
-          <cylinder radius="0.02" length="0.06"/>
-        </geometry>
+        <origin xyz="${coxa_l/2} 0 0" rpy="0 ${pi/2} 0"/>
+        <geometry><cylinder radius="${coxa_r}" length="${coxa_l}"/></geometry>
       </collision>
     </link>
-    <!-- COXA JOINT: revolute around Z, mounted on base sphere surface -->
+    <!-- Coxa joint: on top of base disc, rotates around Z -->
     <joint name="${leg_name}_coxa_joint" type="revolute">
       <parent link="base_link"/>
       <child link="${leg_name}_coxa_link"/>
-      <origin xyz="${hip_x} ${hip_y} ${hip_z}" rpy="0 0 ${hip_yaw}"/>
+      <origin xyz="${hip_x} ${hip_y} ${hip_z_offset}" rpy="0 0 ${hip_yaw}"/>
       <axis xyz="0 0 1"/>
       <limit lower="${-pi/2}" upper="${pi/2}" effort="10.0" velocity="3.14"/>
       <dynamics damping="0.1" friction="0.0"/>
     </joint>
-    <!-- FEMUR LINK -->
-    <!-- Cylinder r=0.018 l=0.12, mass=0.15 kg -->
-    <!-- Oriented along X when joint=0, so cylinder axis is along X (rpy="0 pi/2 0") -->
+    <!-- ── FEMUR LINK ─────────────────────────────────────────────
+         Extends outward+downward from the end of coxa.
+         Axis along X of joint frame (rpy="0 pi/2 0" for visual).
+    ─────────────────────────────────────────────────────────── -->
     <link name="${leg_name}_femur_link">
-      <xacro:cylinder_inertia m="0.15" r="0.018" l="0.12"/>
+      <inertial>
+        <origin xyz="${femur_l/2} 0 0" rpy="0 0 0"/>
+        <mass value="${femur_mass}"/>
+        <inertia
+          ixx="${femur_mass * femur_r*femur_r / 2.0}"
+          iyy="${femur_mass * (3*femur_r*femur_r + femur_l*femur_l) / 12.0}"
+          izz="${femur_mass * (3*femur_r*femur_r + femur_l*femur_l) / 12.0}"
+          ixy="0" ixz="0" iyz="0"/>
+      </inertial>
       <visual>
-        <origin xyz="0.06 0 0" rpy="0 ${pi/2} 0"/>
-        <geometry>
-          <cylinder radius="0.018" length="0.12"/>
-        </geometry>
-        <material name="gray">
-          <color rgba="0.5 0.5 0.5 1.0"/>
-        </material>
+        <origin xyz="${femur_l/2} 0 0" rpy="0 ${pi/2} 0"/>
+        <geometry><cylinder radius="${femur_r}" length="${femur_l}"/></geometry>
+        <material name="link_wood"><color rgba="0.75 0.60 0.35 1.0"/></material>
       </visual>
       <collision>
-        <origin xyz="0.06 0 0" rpy="0 ${pi/2} 0"/>
-        <geometry>
-          <cylinder radius="0.018" length="0.12"/>
-        </geometry>
+        <origin xyz="${femur_l/2} 0 0" rpy="0 ${pi/2} 0"/>
+        <geometry><cylinder radius="${femur_r}" length="${femur_l}"/></geometry>
       </collision>
     </link>
-    <!-- FEMUR JOINT: revolute around Y -->
+    <!-- Femur joint: at end of coxa, rotates around Y -->
+    <!-- rpy="0 -pi/6 0" → femur starts at ~30° downward from horizontal -->
     <joint name="${leg_name}_femur_joint" type="revolute">
       <parent link="${leg_name}_coxa_link"/>
       <child link="${leg_name}_femur_link"/>
-      <origin xyz="0 0 0.06" rpy="0 0 0"/>
+      <origin xyz="${coxa_l} 0 0" rpy="0 ${-pi/6} 0"/>
       <axis xyz="0 1 0"/>
       <limit lower="${-pi/3}" upper="${pi/3}" effort="10.0" velocity="3.14"/>
       <dynamics damping="0.1" friction="0.0"/>
     </joint>
-    <!-- TIBIA LINK -->
-    <!-- Cylinder r=0.015 l=0.15, mass=0.10 kg -->
+    <!-- ── TIBIA LINK ─────────────────────────────────────────────
+         Lower leg, extends further outward+downward.
+         Slightly thinner than femur.
+    ─────────────────────────────────────────────────────────── -->
     <link name="${leg_name}_tibia_link">
-      <xacro:cylinder_inertia m="0.10" r="0.015" l="0.15"/>
+      <inertial>
+        <origin xyz="${tibia_l/2} 0 0" rpy="0 0 0"/>
+        <mass value="${tibia_mass}"/>
+        <inertia
+          ixx="${tibia_mass * tibia_r*tibia_r / 2.0}"
+          iyy="${tibia_mass * (3*tibia_r*tibia_r + tibia_l*tibia_l) / 12.0}"
+          izz="${tibia_mass * (3*tibia_r*tibia_r + tibia_l*tibia_l) / 12.0}"
+          ixy="0" ixz="0" iyz="0"/>
+      </inertial>
       <visual>
-        <origin xyz="0.075 0 0" rpy="0 ${pi/2} 0"/>
-        <geometry>
-          <cylinder radius="0.015" length="0.15"/>
-        </geometry>
-        <material name="light_gray">
-          <color rgba="0.7 0.7 0.7 1.0"/>
-        </material>
+        <origin xyz="${tibia_l/2} 0 0" rpy="0 ${pi/2} 0"/>
+        <geometry><cylinder radius="${tibia_r}" length="${tibia_l}"/></geometry>
+        <material name="link_dark"><color rgba="0.25 0.25 0.25 1.0"/></material>
       </visual>
       <collision>
-        <origin xyz="0.075 0 0" rpy="0 ${pi/2} 0"/>
-        <geometry>
-          <cylinder radius="0.015" length="0.15"/>
-        </geometry>
+        <origin xyz="${tibia_l/2} 0 0" rpy="0 ${pi/2} 0"/>
+        <geometry><cylinder radius="${tibia_r}" length="${tibia_l}"/></geometry>
         <surface>
           <friction>
-            <ode>
-              <mu>1.0</mu>
-              <mu2>1.0</mu2>
-            </ode>
+            <ode><mu>1.0</mu><mu2>1.0</mu2></ode>
           </friction>
         </surface>
       </collision>
     </link>
-    <!-- TIBIA JOINT: revolute around Y -->
+    <!-- Tibia joint: at end of femur, rotates around Y -->
+    <!-- rpy="0 pi/4 0" → tibia starts pointing downward relative to femur -->
     <joint name="${leg_name}_tibia_joint" type="revolute">
       <parent link="${leg_name}_femur_link"/>
       <child link="${leg_name}_tibia_link"/>
-      <origin xyz="0.12 0 0" rpy="0 0 0"/>
+      <origin xyz="${femur_l} 0 0" rpy="0 ${pi/4} 0"/>
       <axis xyz="0 1 0"/>
-      <limit lower="${-2*pi/3}" upper="0" effort="10.0" velocity="3.14"/>
+      <limit lower="${-2*pi/3}" upper="${pi/6}" effort="10.0" velocity="3.14"/>
       <dynamics damping="0.1" friction="0.0"/>
     </joint>
-    <!-- TRANSMISSION: coxa -->
+    <!-- ── TRANSMISSIONS ──────────────────────────────────────── -->
     <transmission name="${leg_name}_coxa_trans">
       <type>transmission_interface/SimpleTransmission</type>
@@ -152,5 +201,4 @@
       </actuator>
     </transmission>
-    <!-- TRANSMISSION: femur -->
     <transmission name="${leg_name}_femur_trans">
       <type>transmission_interface/SimpleTransmission</type>
@@ -163,5 +211,4 @@
       </actuator>
     </transmission>
-    <!-- TRANSMISSION: tibia -->
     <transmission name="${leg_name}_tibia_trans">
       <type>transmission_interface/SimpleTransmission</type>
@@ -176,58 +223,68 @@
   </xacro:macro>
   <!-- ============================================================
-       BASE_FOOTPRINT (virtual ground-plane reference frame)
+       BASE_FOOTPRINT (ground-plane virtual frame)
+       Placed so robot CoM (= base_link z=0) sits at spawn_z above ground.
+       base_footprint is the ground contact reference.
   ============================================================ -->
   <link name="base_footprint"/>
+  <!-- base_link is 0.15 m above base_footprint:
+       base disc half-height (0.0125) + clearance so tibia tips touch ground.
+       Tibia effective reach downward ≈ coxa_l·sin30° + femur_l·sin30° + tibia_l·sin(45°+30°)
+       ≈ 0.0225 + 0.05 + 0.125 ≈ 0.20 m. Use 0.22 m for safety margin. -->
   <joint name="base_footprint_joint" type="fixed">
     <parent link="base_footprint"/>
     <child link="base_link"/>
-    <origin xyz="0 0 0.18" rpy="0 0 0"/>
+    <origin xyz="0 0 0.22" rpy="0 0 0"/>
   </joint>
   <!-- ============================================================
-       BASE_LINK: central sphere
-       r=0.12 m, mass=1.5 kg
-       Inertia (solid sphere): I = 2/5 * 1.5 * 0.12^2 = 0.00864 kg·m²
+       BASE_LINK: flat disc (base) + dome sphere (top)
+       Two visual/collision elements, single inertial (combined CoM at z=0).
   ============================================================ -->
   <link name="base_link">
-    <xacro:sphere_inertia m="1.5" r="0.12"/>
+    <xacro:base_link_inertia/>
+    <!-- Visual 1: flat base disc -->
     <visual>
       <origin xyz="0 0 0" rpy="0 0 0"/>
-      <geometry>
-        <sphere radius="0.12"/>
-      </geometry>
-      <material name="orange">
-        <color rgba="0.9 0.4 0.1 1.0"/>
-      </material>
+      <geometry><cylinder radius="${base_r}" length="${base_h}"/></geometry>
+      <material name="chassis_dark"><color rgba="0.18 0.18 0.20 1.0"/></material>
     </visual>
+    <!-- Visual 2: dome sphere on top -->
+    <visual>
+      <origin xyz="0 0 ${dome_z}" rpy="0 0 0"/>
+      <geometry><sphere radius="${dome_r}"/></geometry>
+      <material name="chassis_orange"><color rgba="0.85 0.35 0.05 1.0"/></material>
+    </visual>
+    <!-- Collision 1: disc -->
     <collision>
       <origin xyz="0 0 0" rpy="0 0 0"/>
-      <geometry>
-        <sphere radius="0.12"/>
-      </geometry>
+      <geometry><cylinder radius="${base_r}" length="${base_h}"/></geometry>
+    </collision>
+    <!-- Collision 2: dome -->
+    <collision>
+      <origin xyz="0 0 ${dome_z}" rpy="0 0 0"/>
+      <geometry><sphere radius="${dome_r}"/></geometry>
     </collision>
   </link>
   <!-- ============================================================
        LEG INSTANTIATION
-       Hip positions on the sphere surface (r=0.12):
-         front_right  ( 45°): x= 0.08485, y= 0.08485
-         front_left   (135°): x=-0.08485, y= 0.08485
-         back_left   (-135°): x=-0.08485, y=-0.08485
-         back_right   (-45°): x= 0.08485, y=-0.08485
-  ============================================================ -->
-  <!-- front_right: hip_yaw = pi/4 = 0.7854 rad -->
+       hip_r = 0.10 m  (radial distance of coxa joint from centre)
+       hip_z = base_h/2 = +0.0125 m  (top surface of base disc)
+       Hip positions (on top face of disc):
+         front_right  ( 45°): x= hip_r·cos45° = 0.07071, y= 0.07071
+         front_left   (135°): x=-0.07071,               y= 0.07071
+         back_left   (-135°): x=-0.07071,               y=-0.07071
+         back_right   (-45°): x= 0.07071,               y=-0.07071
+  ============================================================ -->
   <xacro:leg leg_name="front_right"
-             hip_x="0.08485" hip_y="0.08485" hip_z="0.0"
+             hip_x="0.07071"  hip_y="0.07071"
              hip_yaw="${pi/4}"/>
-  <!-- front_left: hip_yaw = 3*pi/4 = 2.3562 rad -->
   <xacro:leg leg_name="front_left"
-             hip_x="-0.08485" hip_y="0.08485" hip_z="0.0"
+             hip_x="-0.07071" hip_y="0.07071"
              hip_yaw="${3*pi/4}"/>
-  <!-- back_left: hip_yaw = -3*pi/4 = -2.3562 rad -->
   <xacro:leg leg_name="back_left"
-             hip_x="-0.08485" hip_y="-0.08485" hip_z="0.0"
+             hip_x="-0.07071" hip_y="-0.07071"
              hip_yaw="${-3*pi/4}"/>
-  <!-- back_right: hip_yaw = -pi/4 = -0.7854 rad -->
   <xacro:leg leg_name="back_right"
-             hip_x="0.08485" hip_y="-0.08485" hip_z="0.0"
+             hip_x="0.07071"  hip_y="-0.07071"
              hip_yaw="${-pi/4}"/>
   <!-- ============================================================
@@ -241,107 +298,85 @@
     <joint name="front_right_coxa_joint">
       <command_interface name="position">
-        <param name="min">${-pi/2}</param>
-        <param name="max">${pi/2}</param>
-      </command_interface>
-      <state_interface name="position"/>
-      <state_interface name="velocity"/>
+        <param name="min">${-pi/2}</param><param name="max">${pi/2}</param>
+      </command_interface>
+      <state_interface name="position"/><state_interface name="velocity"/>
     </joint>
     <joint name="front_right_femur_joint">
       <command_interface name="position">
-        <param name="min">${-pi/3}</param>
-        <param name="max">${pi/3}</param>
-      </command_interface>
-      <state_interface name="position"/>
-      <state_interface name="velocity"/>
+        <param name="min">${-pi/3}</param><param name="max">${pi/3}</param>
+      </command_interface>
+      <state_interface name="position"/><state_interface name="velocity"/>
     </joint>
     <joint name="front_right_tibia_joint">
       <command_interface name="position">
-        <param name="min">${-2*pi/3}</param>
-        <param name="max">0</param>
-      </command_interface>
-      <state_interface name="position"/>
-      <state_interface name="velocity"/>
+        <param name="min">${-2*pi/3}</param><param name="max">${pi/6}</param>
+      </command_interface>
+      <state_interface name="position"/><state_interface name="velocity"/>
     </joint>
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