Commit message: spider

File: install/spider_description/share/spider_description/urdf/spider.urdf.xacro (robot description, xacro)
@@ -1,23 +1,10 @@
 <?xml version="1.0"?>
 <robot xmlns:xacro="http://www.ros.org/wiki/xacro" name="spider">
-  <!-- ============================================================
-       SPIDER QUADRUPED ROBOT - URDF/XACRO  (Hito 1 rev.3)
-       Body: flat base cylinder + dome mesh (true hemisphere, no clipping)
-       4 legs in X-pattern at 45°/135°/-135°/-45°
-       3 DOF per leg: coxa(Z) → femur(Y) → tibia(Y)
-  ============================================================ -->
-  <!-- ============================================================
-       CONSTANTS
-  ============================================================ -->
-  <!-- Body geometry -->
-  <xacro:property name="base_r"        value="0.12"/>   <!-- base disc radius (wider than dome) -->
-  <xacro:property name="base_h"        value="0.01"/>   <!-- base disc height -->
-  <xacro:property name="dome_r"        value="0.1"/>   <!-- dome mesh radius (hemisphere) -->
-  <!-- dome mesh base sits exactly on top face of disc (z = +base_h/2) -->
+  <xacro:property name="base_r"        value="0.12"/>
+  <xacro:property name="base_h"        value="0.01"/>
+  <xacro:property name="dome_r"        value="0.1"/>
   <xacro:property name="dome_z"        value="${base_h / 2.0}"/>
-  <!-- Hip attachment: on top surface of base disc, at radial distance hip_r -->
-  <xacro:property name="hip_r"         value="${base_r - 0.015}"/>  <!-- radial offset of coxa joint from centre -->
-  <xacro:property name="hip_z_offset"  value="${base_h / 2.0}"/>   <!-- = base_h/2, top of base disc -->
-  <!-- Leg geometry -->
+  <xacro:property name="hip_r"         value="${base_r - 0.015}"/>
+  <xacro:property name="hip_z_offset"  value="${base_h / 2.0}"/>
   <xacro:property name="coxa_r"  value="0.018"/>
   <xacro:property name="coxa_l"  value="0.045"/>
@@ -26,75 +13,35 @@
   <xacro:property name="tibia_r" value="0.012"/>
   <xacro:property name="tibia_l" value="0.13"/>
-  <!-- Masses (total body = 1.5 kg) -->
   <xacro:property name="base_mass"  value="1.5"/>
   <xacro:property name="coxa_mass"  value="0.06"/>
   <xacro:property name="femur_mass" value="0.12"/>
   <xacro:property name="tibia_mass" value="0.08"/>
-  <!-- ============================================================
-       INERTIA MACROS
-  ============================================================ -->
-  <!-- Solid sphere -->
   <xacro:macro name="sphere_inertia" params="m r">
     <inertial>
       <origin xyz="0 0 0" rpy="0 0 0"/>
       <mass value="${m}"/>
-      <inertia
-        ixx="${2.0/5.0 * m * r * r}"
-        iyy="${2.0/5.0 * m * r * r}"
-        izz="${2.0/5.0 * m * r * r}"
-        ixy="0" ixz="0" iyz="0"/>
+      <inertia ixx="${2.0/5.0 * m * r * r}" iyy="${2.0/5.0 * m * r * r}" izz="${2.0/5.0 * m * r * r}" ixy="0" ixz="0" iyz="0"/>
     </inertial>
   </xacro:macro>
-  <!-- Solid cylinder (symmetry axis = Z) -->
   <xacro:macro name="cylinder_inertia" params="m r l">
     <inertial>
       <origin xyz="0 0 0" rpy="0 0 0"/>
       <mass value="${m}"/>
-      <inertia
-        ixx="${m * (3*r*r + l*l) / 12.0}"
-        iyy="${m * (3*r*r + l*l) / 12.0}"
-        izz="${m * r * r / 2.0}"
-        ixy="0" ixz="0" iyz="0"/>
+      <inertia ixx="${m * (3*r*r + l*l) / 12.0}" iyy="${m * (3*r*r + l*l) / 12.0}" izz="${m * r * r / 2.0}" ixy="0" ixz="0" iyz="0"/>
     </inertial>
   </xacro:macro>
-  <!-- Composite inertia for base_link:
-       Modelled as a thick disc (dominant contributor).
-       CoM placed at z=0 (centre of the disc).
-       base_r=0.13  base_h=0.025  m=1.5 kg
-       Ixx=Iyy = m*(3r²+h²)/12  Izz = m*r²/2  -->
   <xacro:macro name="base_link_inertia">
     <inertial>
       <origin xyz="0 0 0" rpy="0 0 0"/>
       <mass value="${base_mass}"/>
-      <inertia
-        ixx="${base_mass * (3*base_r*base_r + base_h*base_h) / 12.0}"
-        iyy="${base_mass * (3*base_r*base_r + base_h*base_h) / 12.0}"
-        izz="${base_mass * base_r*base_r / 2.0}"
-        ixy="0" ixz="0" iyz="0"/>
+      <inertia ixx="${base_mass * (3*base_r*base_r + base_h*base_h) / 12.0}" iyy="${base_mass * (3*base_r*base_r + base_h*base_h) / 12.0}" izz="${base_mass * base_r*base_r / 2.0}" ixy="0" ixz="0" iyz="0"/>
     </inertial>
   </xacro:macro>
-  <!-- ============================================================
-       LEG MACRO
-       hip_x, hip_y : position of the coxa joint in base_link frame
-                       (on top surface of base disc, at the edge)
-       hip_yaw       : yaw angle so coxa extends radially outward
-  ============================================================ -->
   <xacro:macro name="leg" params="leg_name hip_x hip_y hip_yaw">
-    <!-- ── COXA LINK ─────────────────────────────────────────────
-         Small cylinder representing the hip servo block.
-         Oriented radially (axis along X of joint frame).
-         Visual/collision centre at x=coxa_l/2 from joint origin.
-    ─────────────────────────────────────────────────────────── -->
     <link name="${leg_name}_coxa_link">
-      <!-- Inertia: cylinder with axis along X → rotate cylinder_inertia 90° about Y.
-           For a cylinder with axis along X: Ixx=m*r²/2  Iyy=Izz=m*(3r²+l²)/12 -->
       <inertial>
         <origin xyz="${coxa_l/2} 0 0" rpy="0 0 0"/>
         <mass value="${coxa_mass}"/>
-        <inertia
-          ixx="${coxa_mass * coxa_r*coxa_r / 2.0}"
-          iyy="${coxa_mass * (3*coxa_r*coxa_r + coxa_l*coxa_l) / 12.0}"
-          izz="${coxa_mass * (3*coxa_r*coxa_r + coxa_l*coxa_l) / 12.0}"
-          ixy="0" ixz="0" iyz="0"/>
+        <inertia ixx="${coxa_mass * coxa_r*coxa_r / 2.0}" iyy="${coxa_mass * (3*coxa_r*coxa_r + coxa_l*coxa_l) / 12.0}" izz="${coxa_mass * (3*coxa_r*coxa_r + coxa_l*coxa_l) / 12.0}" ixy="0" ixz="0" iyz="0"/>
       </inertial>
       <visual>
@@ -108,5 +55,4 @@
       </collision>
     </link>
-    <!-- Coxa joint: on top of base disc, rotates around Z -->
     <joint name="${leg_name}_coxa_joint" type="revolute">
       <parent link="base_link"/>
@@ -117,17 +63,9 @@
       <dynamics damping="0.1" friction="0.0"/>
     </joint>
-    <!-- ── FEMUR LINK ─────────────────────────────────────────────
-         Extends outward+downward from the end of coxa.
-         Axis along X of joint frame (rpy="0 pi/2 0" for visual).
-    ─────────────────────────────────────────────────────────── -->
     <link name="${leg_name}_femur_link">
       <inertial>
         <origin xyz="${femur_l/2} 0 0" rpy="0 0 0"/>
         <mass value="${femur_mass}"/>
-        <inertia
-          ixx="${femur_mass * femur_r*femur_r / 2.0}"
-          iyy="${femur_mass * (3*femur_r*femur_r + femur_l*femur_l) / 12.0}"
-          izz="${femur_mass * (3*femur_r*femur_r + femur_l*femur_l) / 12.0}"
-          ixy="0" ixz="0" iyz="0"/>
+        <inertia ixx="${femur_mass * femur_r*femur_r / 2.0}" iyy="${femur_mass * (3*femur_r*femur_r + femur_l*femur_l) / 12.0}" izz="${femur_mass * (3*femur_r*femur_r + femur_l*femur_l) / 12.0}" ixy="0" ixz="0" iyz="0"/>
       </inertial>
       <visual>
@@ -141,6 +79,4 @@
       </collision>
     </link>
-    <!-- Femur joint: at end of coxa, rotates around Y -->
-    <!-- rpy="0 -pi/6 0" → femur starts at ~30° downward from horizontal -->
     <joint name="${leg_name}_femur_joint" type="revolute">
       <parent link="${leg_name}_coxa_link"/>
@@ -151,17 +87,9 @@
       <dynamics damping="0.1" friction="0.0"/>
     </joint>
-    <!-- ── TIBIA LINK ─────────────────────────────────────────────
-         Lower leg, extends further outward+downward.
-         Slightly thinner than femur.
-    ─────────────────────────────────────────────────────────── -->
     <link name="${leg_name}_tibia_link">
       <inertial>
         <origin xyz="${tibia_l/2} 0 0" rpy="0 0 0"/>
         <mass value="${tibia_mass}"/>
-        <inertia
-          ixx="${tibia_mass * tibia_r*tibia_r / 2.0}"
-          iyy="${tibia_mass * (3*tibia_r*tibia_r + tibia_l*tibia_l) / 12.0}"
-          izz="${tibia_mass * (3*tibia_r*tibia_r + tibia_l*tibia_l) / 12.0}"
-          ixy="0" ixz="0" iyz="0"/>
+        <inertia ixx="${tibia_mass * tibia_r*tibia_r / 2.0}" iyy="${tibia_mass * (3*tibia_r*tibia_r + tibia_l*tibia_l) / 12.0}" izz="${tibia_mass * (3*tibia_r*tibia_r + tibia_l*tibia_l) / 12.0}" ixy="0" ixz="0" iyz="0"/>
       </inertial>
       <visual>
@@ -173,23 +101,10 @@
         <origin xyz="${tibia_l/2} 0 0" rpy="0 ${pi/2} 0"/>
         <geometry><cylinder radius="${tibia_r}" length="${tibia_l}"/></geometry>
-        <surface>
-          <friction>
-            <ode><mu>1.0</mu><mu2>1.0</mu2></ode>
-          </friction>
-        </surface>
       </collision>
-      <!-- Foot-tip sphere: point contact at the end of the tibia for better ground grip -->
       <collision>
         <origin xyz="${tibia_l} 0 0" rpy="0 0 0"/>
         <geometry><sphere radius="${tibia_r}"/></geometry>
-        <surface>
-          <friction>
-            <ode><mu>1.0</mu><mu2>1.0</mu2></ode>
-          </friction>
-        </surface>
       </collision>
     </link>
-    <!-- Tibia joint: at end of femur, rotates around Y -->
-    <!-- rpy="0 pi/4 0" → tibia starts pointing downward relative to femur -->
     <joint name="${leg_name}_tibia_joint" type="revolute">
       <parent link="${leg_name}_femur_link"/>
@@ -197,49 +112,12 @@
       <origin xyz="${femur_l} 0 0" rpy="0 ${pi/4} 0"/>
       <axis xyz="0 1 0"/>
-      <limit lower="${-2*pi/3}" upper="${pi/6}" effort="10.0" velocity="3.14"/>
+      <limit lower="${-pi/2}" upper="${pi/2}" effort="10.0" velocity="3.14"/>
       <dynamics damping="0.1" friction="0.0"/>
     </joint>
-    <!-- ── TRANSMISSIONS ──────────────────────────────────────── -->
-    <transmission name="${leg_name}_coxa_trans">
-      <type>transmission_interface/SimpleTransmission</type>
-      <joint name="${leg_name}_coxa_joint">
-        <hardwareInterface>hardware_interface/PositionJointInterface</hardwareInterface>
-      </joint>
-      <actuator name="${leg_name}_coxa_joint_motor">
-        <hardwareInterface>hardware_interface/PositionJointInterface</hardwareInterface>
-        <mechanicalReduction>1</mechanicalReduction>
-      </actuator>
-    </transmission>
-    <transmission name="${leg_name}_femur_trans">
-      <type>transmission_interface/SimpleTransmission</type>
-      <joint name="${leg_name}_femur_joint">
-        <hardwareInterface>hardware_interface/PositionJointInterface</hardwareInterface>
-      </joint>
-      <actuator name="${leg_name}_femur_joint_motor">
-        <hardwareInterface>hardware_interface/PositionJointInterface</hardwareInterface>
-        <mechanicalReduction>1</mechanicalReduction>
-      </actuator>
-    </transmission>
-    <transmission name="${leg_name}_tibia_trans">
-      <type>transmission_interface/SimpleTransmission</type>
-      <joint name="${leg_name}_tibia_joint">
-        <hardwareInterface>hardware_interface/PositionJointInterface</hardwareInterface>
-      </joint>
-      <actuator name="${leg_name}_tibia_joint_motor">
-        <hardwareInterface>hardware_interface/PositionJointInterface</hardwareInterface>
-        <mechanicalReduction>1</mechanicalReduction>
-      </actuator>
-    </transmission>
+    <transmission name="${leg_name}_coxa_trans"><type>transmission_interface/SimpleTransmission</type><joint name="${leg_name}_coxa_joint"><hardwareInterface>hardware_interface/PositionJointInterface</hardwareInterface></joint><actuator name="${leg_name}_coxa_joint_motor"><hardwareInterface>hardware_interface/PositionJointInterface</hardwareInterface><mechanicalReduction>1</mechanicalReduction></actuator></transmission>
+    <transmission name="${leg_name}_femur_trans"><type>transmission_interface/SimpleTransmission</type><joint name="${leg_name}_femur_joint"><hardwareInterface>hardware_interface/PositionJointInterface</hardwareInterface></joint><actuator name="${leg_name}_femur_joint_motor"><hardwareInterface>hardware_interface/PositionJointInterface</hardwareInterface><mechanicalReduction>1</mechanicalReduction></actuator></transmission>
+    <transmission name="${leg_name}_tibia_trans"><type>transmission_interface/SimpleTransmission</type><joint name="${leg_name}_tibia_joint"><hardwareInterface>hardware_interface/PositionJointInterface</hardwareInterface></joint><actuator name="${leg_name}_tibia_joint_motor"><hardwareInterface>hardware_interface/PositionJointInterface</hardwareInterface><mechanicalReduction>1</mechanicalReduction></actuator></transmission>
   </xacro:macro>
-  <!-- ============================================================
-       BASE_FOOTPRINT (ground-plane virtual frame)
-       Placed so robot CoM (= base_link z=0) sits at spawn_z above ground.
-       base_footprint is the ground contact reference.
-  ============================================================ -->
   <link name="base_footprint"/>
-  <!-- base_link is 0.15 m above base_footprint:
-       base disc half-height (0.0125) + clearance so tibia tips touch ground.
-       Tibia effective reach downward ≈ coxa_l·sin30° + femur_l·sin30° + tibia_l·sin(45°+30°)
-       ≈ 0.0225 + 0.05 + 0.125 ≈ 0.20 m. Use 0.22 m for safety margin. -->
   <joint name="base_footprint_joint" type="fixed">
     <parent link="base_footprint"/>
@@ -247,11 +125,6 @@
     <origin xyz="0 0 0.30" rpy="0 0 0"/>
   </joint>
-  <!-- ============================================================
-       BASE_LINK: flat disc (base) + dome sphere (top)
-       Two visual/collision elements, single inertial (combined CoM at z=0).
-  ============================================================ -->
   <link name="base_link">
     <xacro:base_link_inertia/>
-    <!-- Visual 1: flat base disc -->
     <visual>
       <origin xyz="0 0 0" rpy="0 0 0"/>
@@ -259,19 +132,13 @@
       <material name="chassis_dark"><color rgba="0.18 0.18 0.20 1.0"/></material>
     </visual>
-    <!-- Visual 2: dome mesh (true hemisphere, base flat at Z=0 in mesh space) -->
     <visual>
       <origin xyz="0 0 ${dome_z}" rpy="0 0 0"/>
-      <geometry>
-        <mesh filename="package://spider_description/meshes/dome.obj"/>
-      </geometry>
+      <geometry><mesh filename="package://spider_description/meshes/dome.obj"/></geometry>
       <material name="chassis_orange"><color rgba="0.85 0.35 0.05 1.0"/></material>
     </visual>
-    <!-- Collision 1: disc -->
     <collision>
       <origin xyz="0 0 0" rpy="0 0 0"/>
       <geometry><cylinder radius="${base_r}" length="${base_h}"/></geometry>
     </collision>
-    <!-- Collision 2: dome approximated as cylinder (r=dome_r, h=dome_r) -->
-    <!-- Cylinder center at z = dome_z + dome_r/2 to cover the dome volume -->
     <collision>
       <origin xyz="0 0 ${dome_z + dome_r/2.0}" rpy="0 0 0"/>
@@ -279,158 +146,38 @@
     </collision>
   </link>
-  <!-- ============================================================
-       LEG INSTANTIATION
-       hip_r = base_r - 0.015  (radial distance of coxa joint from centre)
-       hip_z = base_h/2        (top surface of base disc)
-       Hip positions (on top face of disc):
-         front_right  ( 45°): x= hip_r·cos45°, y= hip_r·sin45°
-         front_left   (135°): x=-hip_r·cos45°, y= hip_r·sin45°
-         back_left   (-135°): x=-hip_r·cos45°, y=-hip_r·sin45°
-         back_right   (-45°): x= hip_r·cos45°, y=-hip_r·sin45°
-  ============================================================ -->
-  <xacro:leg leg_name="front_right"
-             hip_x="${hip_r * 0.70711}"  hip_y="${hip_r * 0.70711}"
-             hip_yaw="${pi/4}"/>
-  <xacro:leg leg_name="front_left"
-             hip_x="${-hip_r * 0.70711}" hip_y="${hip_r * 0.70711}"
-             hip_yaw="${3*pi/4}"/>
-  <xacro:leg leg_name="back_left"
-             hip_x="${-hip_r * 0.70711}" hip_y="${-hip_r * 0.70711}"
-             hip_yaw="${-3*pi/4}"/>
-  <xacro:leg leg_name="back_right"
-             hip_x="${hip_r * 0.70711}"  hip_y="${-hip_r * 0.70711}"
-             hip_yaw="${-pi/4}"/>
-  <!-- ============================================================
-       ROS2_CONTROL HARDWARE INTERFACE
-  ============================================================ -->
+  <xacro:leg leg_name="front_right" hip_x="${hip_r * 0.70711}"  hip_y="${hip_r * 0.70711}" hip_yaw="${pi/4}"/>
+  <xacro:leg leg_name="front_left"  hip_x="${-hip_r * 0.70711}" hip_y="${hip_r * 0.70711}" hip_yaw="${3*pi/4}"/>
+  <xacro:leg leg_name="back_left"   hip_x="${-hip_r * 0.70711}" hip_y="${-hip_r * 0.70711}" hip_yaw="${-3*pi/4}"/>
+  <xacro:leg leg_name="back_right"  hip_x="${hip_r * 0.70711}"  hip_y="${-hip_r * 0.70711}" hip_yaw="${-pi/4}"/>
   <ros2_control name="spider_ign_ros2_control" type="system">
     <hardware>
       <plugin>ign_ros2_control/IgnitionSystem</plugin>
     </hardware>
-    <!-- front_right -->
-    <joint name="front_right_coxa_joint">
-      <command_interface name="position">
-        <param name="min">${-pi/2}</param><param name="max">${pi/2}</param>
-        <param name="p">100.0</param>
-        <param name="i">0.1</param>
-        <param name="d">1.0</param>
-      </command_interface>
-      <state_interface name="position"/><state_interface name="velocity"/>
-    </joint>
-    <joint name="front_right_femur_joint">
-      <command_interface name="position">
-        <param name="min">${-pi/3}</param><param name="max">${pi/3}</param>
-        <param name="p">100.0</param>
-        <param name="i">0.1</param>
-        <param name="d">1.0</param>
-      </command_interface>
-      <state_interface name="position"/><state_interface name="velocity"/>
-    </joint>
-    <joint name="front_right_tibia_joint">
-      <command_interface name="position">
-        <param name="min">${-2*pi/3}</param><param name="max">${pi/6}</param>
-        <param name="p">100.0</param>
-        <param name="i">0.1</param>
-        <param name="d">1.0</param>
-      </command_interface>
-      <state_interface name="position"/><state_interface name="velocity"/>
-    </joint>
-    <!-- front_left -->
-    <joint name="front_left_coxa_joint">
-      <command_interface name="position">
-        <param name="min">${-pi/2}</param><param name="max">${pi/2}</param>
-        <param name="p">100.0</param>
-        <param name="i">0.1</param>
-        <param name="d">1.0</param>
-      </command_interface>
-      <state_interface name="position"/><state_interface name="velocity"/>
-    </joint>
-    <joint name="front_left_femur_joint">
-      <command_interface name="position">
-        <param name="min">${-pi/3}</param><param name="max">${pi/3}</param>
-        <param name="p">100.0</param>
-        <param name="i">0.1</param>
-        <param name="d">1.0</param>
-      </command_interface>
-      <state_interface name="position"/><state_interface name="velocity"/>
-    </joint>
-    <joint name="front_left_tibia_joint">
-      <command_interface name="position">
-        <param name="min">${-2*pi/3}</param><param name="max">${pi/6}</param>
-        <param name="p">100.0</param>
-        <param name="i">0.1</param>
-        <param name="d">1.0</param>
-      </command_interface>
-      <state_interface name="position"/><state_interface name="velocity"/>
-    </joint>
-    <!-- back_left -->
-    <joint name="back_left_coxa_joint">
-      <command_interface name="position">
-        <param name="min">${-pi/2}</param><param name="max">${pi/2}</param>
-        <param name="p">100.0</param>
-        <param name="i">0.1</param>
-        <param name="d">1.0</param>
-      </command_interface>
-      <state_interface name="position"/><state_interface name="velocity"/>
-    </joint>
-    <joint name="back_left_femur_joint">
-      <command_interface name="position">
-        <param name="min">${-pi/3}</param><param name="max">${pi/3}</param>
-        <param name="p">100.0</param>
-        <param name="i">0.1</param>
-        <param name="d">1.0</param>
-      </command_interface>
-      <state_interface name="position"/><state_interface name="velocity"/>
-    </joint>
-    <joint name="back_left_tibia_joint">
-      <command_interface name="position">
-        <param name="min">${-2*pi/3}</param><param name="max">${pi/6}</param>
-        <param name="p">100.0</param>
-        <param name="i">0.1</param>
-        <param name="d">1.0</param>
-      </command_interface>
-      <state_interface name="position"/><state_interface name="velocity"/>
-    </joint>
-    <!-- back_right -->
-    <joint name="back_right_coxa_joint">
-      <command_interface name="position">
-        <param name="min">${-pi/2}</param><param name="max">${pi/2}</param>
-        <param name="p">100.0</param>
-        <param name="i">0.1</param>
-        <param name="d">1.0</param>
-      </command_interface>
-      <state_interface name="position"/><state_interface name="velocity"/>
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